Commit message: camera position

File: urdf/camera.urdf.xacro (robot description, xacro)
@@ -25,5 +25,5 @@
         </link>
         <joint name="camera_joint" type="fixed">
-            <origin xyz="0.081 0.0 0.1125" rpy="0 0 0" />
+            <origin xyz="0.081 0.0 0.1125" rpy="0 0.3 0" />
             <parent link="base_link" />
             <child link="camera_link" />
