Commit message: change colors

File: urdf/tcebot.urdf.xacro (robot description, xacro)
@@ -14,5 +14,5 @@
         <mesh filename="package://tcebot_description/meshes/base_link.stl" scale="0.001 0.001 0.001" />
       </geometry>
-      <material name="silver" />
+      <material name="light_blue" />
     </visual>
     <collision>
@@ -35,5 +35,5 @@
           scale="0.001 0.001 0.001" />
       </geometry>
-      <material name="black" />
+      <material name="dark_grey" />
     </visual>
     <collision>
@@ -57,5 +57,5 @@
           scale="0.001 0.001 0.001" />
       </geometry>
-      <material name="black" />
+      <material name="dark_grey" />
     </visual>
     <collision>
@@ -78,5 +78,5 @@
         <mesh filename="package://tcebot_description/meshes/lidar.stl" scale="0.001 0.001 0.001" />
       </geometry>
-      <material name="light_blue" />
+      <material name="dark_grey" />
     </visual>
     <collision>

Commit message: wheel orientation change

File: urdf/tcebot.urdf.xacro (robot description, xacro)
@@ -112,5 +112,5 @@
     <parent link="base_link" />
     <child link="left_wheel" />
-    <axis xyz="1.0 0.0 0.0" />
+    <axis xyz="0.1 0.0 0.0" />
   </joint>
   <joint name="right_motor" type="continuous">
@@ -118,5 +118,5 @@
     <parent link="base_link" />
     <child link="right_wheel" />
-    <axis xyz="-1.0 0.0 0.0" />
+    <axis xyz="0.1 0.0 0.0" />
   </joint>
   <joint name="rigid1" type="fixed">

Commit message: updates

File: urdf/tcebot.urdf.xacro (robot description, xacro)
@@ -67,4 +67,24 @@
     </collision>
   </link>
+  <link name="caster">
+    <inertial>
+      <origin xyz="8.760371028013886e-06 -0.015006453046049681 -0.008779771570198129" rpy="0 0 0"/>
+      <mass value="0.02176904247885505"/>
+      <inertia ixx="1e-06" iyy="1e-06" izz="1e-06" ixy="-0.0" iyz="0.0" ixz="-0.0"/>
+    </inertial>
+    <visual>
+      <origin xyz="0.008206 -0.049407 -0.007659" rpy="0 0 0"/>
+      <geometry>
+       <mesh filename="package://tcebot_description/meshes/caster.stl" scale="0.001 0.001 0.001"/>
+      </geometry>
+      <material name="silver"/>
+    </visual>
+    <collision>
+      <origin xyz="0.008206 -0.049407 -0.007659" rpy="0 0 0"/>
+      <geometry>
+       <mesh filename="package://tcebot_description/meshes/caster.stl" scale="0.001 0.001 0.001"/>
+      </geometry>
+  </collision>
+  </link>
   <link name="lidar">
     <inertial>
@@ -130,3 +150,10 @@
     <child link="camera" />
   </joint>
+  <joint name="rigid3" type="fixed">
+    <origin xyz="-0.008206 0.049407 0.007659" rpy="0 0 0"/>
+    <parent link="base_link"/>
+    <child link="caster"/>
+    <axis xyz="0 0 1" />
+    <dynamics damping="0.01" friction="0.0"/>
+  </joint>
 </robot>

Commit message: bug fixes

File: urdf/tcebot.urdf.xacro (robot description, xacro)
@@ -4,13 +4,14 @@
   <link name="base_link">
     <inertial>
-      <origin xyz="-0.008564396962539625 -0.014118727809814683 0.06971558782741398" rpy="0 0 0" />
-      <mass value="2.6923940926278465" />
-      <inertia ixx="0.009628" iyy="0.007653" izz="0.007608" ixy="-9e-06" iyz="0.000253"
-        ixz="-1.3e-05" />
+      <origin xyz="-0.008567887520232373 -0.013246764867535883 0.07017948094061893" rpy="0 0 0" />
+      <mass value="2.67513576192234" />
+      <inertia ixx="0.009344" iyy="0.007563" izz="0.007414" ixy="-1e-05" iyz="0.000344"
+        ixz="-1.4e-05" />
     </inertial>
     <visual>
       <origin xyz="0 0 0" rpy="0 0 0" />
       <geometry>
-        <mesh filename="package://tcebot_description/meshes/base_link.stl" scale="0.001 0.001 0.001" />
+        <mesh filename="package://tcebot_description/meshes/base_link.stl"
+          scale="0.001 0.001 0.001" />
       </geometry>
       <material name="light_blue" />
@@ -19,16 +20,17 @@
       <origin xyz="0 0 0" rpy="0 0 0" />
       <geometry>
-        <mesh filename="package://tcebot_description/meshes/base_link.stl" scale="0.001 0.001 0.001" />
+        <mesh filename="package://tcebot_description/meshes/base_link.stl"
+          scale="0.001 0.001 0.001" />
       </geometry>
     </collision>
   </link>
-  <link name="left_wheel">
+  <link name="left_wheel_link">
     <inertial>
-      <origin xyz="-0.015689995537150135 1.9354447389208218e-07 -1.8592013856927325e-07" rpy="0 0 0" />
+      <origin xyz="-0.015689995537150135 1.9354447388514329e-07 -1.8592013858315104e-07" rpy="0 0 0" />
       <mass value="0.23341302374486034" />
       <inertia ixx="0.00016" iyy="9.6e-05" izz="9.6e-05" ixy="0.0" iyz="-0.0" ixz="0.0" />
     </inertial>
     <visual>
-      <origin xyz="0.045157 0.069525 -0.021641" rpy="0 0 0" />
+      <origin xyz="0.045157 0.054525 -0.021641" rpy="0 0 0" />
       <geometry>
         <mesh filename="package://tcebot_description/meshes/left_wheel.stl"
@@ -38,5 +40,5 @@
     </visual>
     <collision>
-      <origin xyz="0.045157 0.069525 -0.021641" rpy="0 0 0" />
+      <origin xyz="0.045157 0.054525 -0.021641" rpy="0 0 0" />
       <geometry>
         <mesh filename="package://tcebot_description/meshes/left_wheel.stl"
@@ -45,12 +47,12 @@
     </collision>
   </link>
-  <link name="right_wheel">
+  <link name="right_wheel_link">
     <inertial>
-      <origin xyz="0.014689947615311807 1.9270939681514943e-07 -6.875961525952545e-07" rpy="0 0 0" />
-      <mass value="0.23341306478013937" />
+      <origin xyz="0.014689947615311793 1.9270939682208832e-07 -6.875961526091323e-07" rpy="0 0 0" />
+      <mass value="0.2334130647801394" />
       <inertia ixx="0.00016" iyy="9.6e-05" izz="9.6e-05" ixy="-0.0" iyz="0.0" ixz="0.0" />
     </inertial>
     <visual>
-      <origin xyz="-0.030621 0.069525 -0.021641" rpy="0 0 0" />
+      <origin xyz="-0.030621 0.054525 -0.021641" rpy="0 0 0" />
       <geometry>
         <mesh filename="package://tcebot_description/meshes/right_wheel.stl"
@@ -60,5 +62,5 @@
     </visual>
     <collision>
-      <origin xyz="-0.030621 0.069525 -0.021641" rpy="0 0 0" />
+      <origin xyz="-0.030621 0.054525 -0.021641" rpy="0 0 0" />
       <geometry>
         <mesh filename="package://tcebot_description/meshes/right_wheel.stl"
@@ -67,27 +69,7 @@
     </collision>
   </link>
-  <link name="caster">
+  <link name="rplidar_link">
     <inertial>
-      <origin xyz="8.760371028013886e-06 -0.015006453046049681 -0.008779771570198129" rpy="0 0 0"/>
-      <mass value="0.02176904247885505"/>
-      <inertia ixx="1e-06" iyy="1e-06" izz="1e-06" ixy="-0.0" iyz="0.0" ixz="-0.0"/>
-    </inertial>
-    <visual>
-      <origin xyz="0.008206 -0.049407 -0.007659" rpy="0 0 0"/>
-      <geometry>
-       <mesh filename="package://tcebot_description/meshes/caster.stl" scale="0.001 0.001 0.001"/>
-      </geometry>
-      <material name="silver"/>
-    </visual>
-    <collision>
-      <origin xyz="0.008206 -0.049407 -0.007659" rpy="0 0 0"/>
-      <geometry>
-       <mesh filename="package://tcebot_description/meshes/caster.stl" scale="0.001 0.001 0.001"/>
-      </geometry>
-  </collision>
-  </link>
-  <link name="lidar">
-    <inertial>
-      <origin xyz="0.01253399240967995 0.034954225501993154 0.031144245322156733" rpy="0 0 0" />
+      <origin xyz="0.012533992409679966 0.034954225501993154 0.031144245322156733" rpy="0 0 0" />
       <mass value="0.5204475795482929" />
       <inertia ixx="0.00026" iyy="0.000181" izz="0.000381" ixy="3e-06" iyz="-2.3e-05" ixz="2e-06" />
@@ -96,5 +78,6 @@
       <origin xyz="0.024795 0.052459 -0.139659" rpy="0 0 0" />
       <geometry>
-        <mesh filename="package://tcebot_description/meshes/lidar.stl" scale="0.001 0.001 0.001" />
+        <mesh filename="package://tcebot_description/meshes/lidar.stl"
+          scale="0.001 0.001 0.001" />
       </geometry>
       <material name="dark_grey" />
@@ -103,9 +86,10 @@
       <origin xyz="0.024795 0.052459 -0.139659" rpy="0 0 0" />
       <geometry>
-        <mesh filename="package://tcebot_description/meshes/lidar.stl" scale="0.001 0.001 0.001" />
+        <mesh filename="package://tcebot_description/meshes/lidar.stl"
+          scale="0.001 0.001 0.001" />
       </geometry>
     </collision>
   </link>
-  <link name="camera">
+  <link name="camera_link">
     <inertial>
       <origin xyz="-8.673617379884035e-18 -0.0015001643555897087 -3.9943743584958114e-07"
@@ -117,5 +101,6 @@
       <origin xyz="0.008 0.091056 -0.138159" rpy="0 0 0" />
       <geometry>
-        <mesh filename="package://tcebot_description/meshes/camera.stl" scale="0.001 0.001 0.001" />
+        <mesh filename="package://tcebot_description/meshes/camera.stl"
+          scale="0.001 0.001 0.001" />
       </geometry>
       <material name="yellow" />
@@ -124,36 +109,61 @@
       <origin xyz="0.008 0.091056 -0.138159" rpy="0 0 0" />
       <geometry>
-        <mesh filename="package://tcebot_description/meshes/camera.stl" scale="0.001 0.001 0.001" />
+        <mesh filename="package://tcebot_description/meshes/camera.stl"
+          scale="0.001 0.001 0.001" />
       </geometry>
     </collision>
   </link>
-  <joint name="left_motor" type="continuous">
-    <origin xyz="-0.045157 -0.069525 0.021641" rpy="0 0 0" />
+  <link name="caster_link">
+    <inertial>
+      <origin xyz="8.760371028013886e-06 -0.015006453046049681 -0.008779771570198129" rpy="0 0 0" />
+      <mass value="0.02176904247885505" />
+      <inertia ixx="1e-06" iyy="1e-06" izz="1e-06" ixy="-0.0" iyz="0.0" ixz="-0.0" />
+    </inertial>
+    <visual>
+      <origin xyz="0.008206 -0.049407 -0.007659" rpy="0 0 0" />
+      <geometry>
+        <mesh filename="package://tcebot_description/meshes/caster.stl"
+          scale="0.001 0.001 0.001" />
+      </geometry>
+      <material name="silver" />
+    </visual>
+    <collision>
+      <origin xyz="0.008206 -0.049407 -0.007659" rpy="0 0 0" />
+      <geometry>
+        <mesh filename="package://tcebot_description/meshes/caster.stl"
+          scale="0.001 0.001 0.001" />
+      </geometry>
+    </collision>
+  </link>
+  <joint name="left_wheel_joint" type="continuous">
+    <origin xyz="-0.045157 -0.054525 0.021641" rpy="0 0 0" />
     <parent link="base_link" />
-    <child link="left_wheel" />
-    <axis xyz="0.1 0.0 0.0" />
+    <child link="left_wheel_link" />
+    <axis xyz="1.0 0.0 0.0" />
+    <dynamics damping="0.01" friction="0.0"/>
   </joint>
-  <joint name="right_motor" type="continuous">
-    <origin xyz="0.030621 -0.069525 0.021641" rpy="0 0 0" />
+  <joint name="right_wheel_joint" type="continuous">
+    <origin xyz="0.030621 -0.054525 0.021641" rpy="0 0 0" />
     <parent link="base_link" />
-    <child link="right_wheel" />
-    <axis xyz="0.1 0.0 0.0" />
+    <child link="right_wheel_link" />
+    <axis xyz="1.0 0.0 0.0" />
+    <dynamics damping="0.01" friction="0.0"/>
   </joint>
-  <joint name="rigid1" type="fixed">
+  <joint name="lidar_joint" type="fixed">
     <origin xyz="-0.024795 -0.052459 0.139659" rpy="0 0 0" />
     <parent link="base_link" />
-    <child link="lidar" />
+    <child link="rplidar_link" />
   </joint>
-  <joint name="rigid2" type="fixed">
+  <joint name="camera_joint" type="fixed">
     <origin xyz="-0.008 -0.091056 0.138159" rpy="0 0 0" />
     <parent link="base_link" />
-    <child link="camera" />
+    <child link="camera_link" />
   </joint>
-  <joint name="rigid3" type="fixed">
-    <origin xyz="-0.008206 0.049407 0.007659" rpy="0 0 0"/>
-    <parent link="base_link"/>
-    <child link="caster"/>
+  <joint name="caster_joint" type="fixed">
+    <origin xyz="-0.008206 0.049407 0.007659" rpy="0 0 0" />
+    <parent link="base_link" />
+    <child link="caster_link" />
     <axis xyz="0 0 1" />
-    <dynamics damping="0.01" friction="0.0"/>
+    <dynamics damping="0.01" friction="0.0" />
   </joint>
 </robot>

Commit message: imu link

File: urdf/tcebot.urdf.xacro (robot description, xacro)
@@ -1,4 +1,5 @@
 <?xml version="1.0"?>
-<robot name="tcebot" xmlns:xacro="http://ros.org/wiki/xacro">
+<robot name="tcebot"
+  xmlns:xacro="http://ros.org/wiki/xacro">
   <xacro:include filename="$(find tcebot_description)/urdf/common_properties.urdf.xacro" />
   <xacro:include filename="$(find tcebot_description)/urdf/wheel_right.urdf.xacro" />
@@ -12,6 +13,5 @@
   <link name="base_link">
     <inertial>
-      <origin xyz="-0.01345975744118259 9.019950050370612e-13 0.061742047216749814"
-        rpy="0 0 0" />
+      <origin xyz="-0.01345975744118259 9.019950050370612e-13 0.061742047216749814" rpy="0 0 0" />
       <mass value="2.49172678848136" />
       <inertia ixx="0.00765" iyy="0.008487" izz="0.007523" ixy="-0.0" iyz="0.0" ixz="0.000145" />
@@ -20,6 +20,5 @@
       <origin xyz="0 0 0" rpy="0 0 0" />
       <geometry>
-        <mesh filename="package://tcebot_description/meshes/base_link.stl"
-          scale="0.001 0.001 0.001" />
+        <mesh filename="package://tcebot_description/meshes/base_link.stl" scale="0.001 0.001 0.001" />
       </geometry>
     </visual>
@@ -27,9 +26,37 @@
       <origin xyz="0 0 0" rpy="0 0 0" />
       <geometry>
-        <mesh filename="package://tcebot_description/meshes/base_link.stl"
-          scale="0.001 0.001 0.001" />
+        <mesh filename="package://tcebot_description/meshes/base_link.stl" scale="0.001 0.001 0.001" />
       </geometry>
     </collision>
   </link>
+  <!-- IMU Link -->
+  <link name="imu_link">
+    <inertial>
+      <origin xyz="0 0 0" rpy="0 0 0" />
+      <mass value="0.05" />
+      <inertia ixx="0.000001" iyy="0.000001" izz="0.000001" ixy="0.0" iyz="0.0" ixz="0.0" />
+    </inertial>
+    <visual>
+      <origin xyz="0 0 0" rpy="0 0 0" />
+      <geometry>
+        <box size="0.02 0.02 0.01" />
+      </geometry>
+      <material name="blue">
+        <color rgba="0.0 0.0 1.0 1.0"/>
+      </material>
+    </visual>
+    <collision>
+      <origin xyz="0 0 0" rpy="0 0 0" />
+      <geometry>
+        <box size="0.02 0.02 0.01" />
+      </geometry>
+    </collision>
+  </link>
+  <!-- IMU Joint (Fixed to Base Link) -->
+  <joint name="imu_joint" type="fixed">
+    <parent link="base_link"/>
+    <child link="imu_link"/>
+    <origin xyz="0 0 0.1" rpy="0 0 0"/>
+  </joint>
   <xacro:wheel_right gazebo="$(arg gazebo)" />
   <xacro:wheel_left gazebo="$(arg gazebo)" />
@@ -46,7 +73,5 @@
   </gazebo>
   <gazebo>
-    <plugin
-      filename="gz-sim-diff-drive-system"
-      name="gz::sim::systems::DiffDrive">
+    <plugin filename="gz-sim-diff-drive-system" name="gz::sim::systems::DiffDrive">
       <left_joint>left_wheel_joint</left_joint>
       <right_joint>right_wheel_joint</right_joint>
@@ -68,7 +93,5 @@
       <odom_publish_frequency>30</odom_publish_frequency>
     </plugin>
-    <plugin
-      filename="gz-sim-joint-state-publisher-system"
-      name="gz::sim::systems::JointStatePublisher">
+    <plugin filename="gz-sim-joint-state-publisher-system" name="gz::sim::systems::JointStatePublisher">
       <joint_name>left_wheel_joint</joint_name>
       <joint_name>right_wheel_joint</joint_name>
@@ -76,4 +99,15 @@
       <update_rate>30</update_rate>
     </plugin>
+    <!-- IMU Sensor Plugin -->
+    <plugin filename="gz-sim-imu-sensor-system" name="gz::sim::systems::ImuSensor">
+      <sensor_name>imu_sensor</sensor_name>
+      <topic>/imu</topic>
+      <update_rate>50</update_rate>
+      <parent_frame>imu_link</parent_frame>
+      <child_frame>base_link</child_frame>
+      <orientation>true</orientation>
+      <angular_velocity>true</angular_velocity>
+      <linear_acceleration>true</linear_acceleration>
+    </plugin>
   </gazebo>
 </robot>
